File: ProPrj_Maggy 4.1_2025-02-07.kicad_sch (KiCad schematic)
At the start: 75 parts, among them CN1 0430450800, CN2 430451000, U1 A4950ELJTR-T, U10 A4950ELJTR-T, U11 LM1117S-5.0, U12 LM1117S-3.3, U13 TLV2372IDR, U15 INA214AIDCKR, U16 INA214AIDCKR, U18 INA214AIDCKR, U19 INA214AIDCKR, U2 A4950ELJTR-T, U20 TMAG5170A2DGKR, U21 TMAG5170A2DGKR, U22 TMAG5170A2DGKR, U23 TMAG5170A2DGKR, U24 TMAG5170A2DGKR, U25 Socket for Teensy 4.1 (2x 1x2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, U3 CH224K, U4 BZT52C6V2, U5 XY308-2.54-2P, U6 XY308-2.54-2P, U7 XY308-2.54-2P, U8 XY308-2.54-2P, U9 A4950ELJTR-T

Commit message: chore: replaced more easyeda components with KiCad counterparts
Components: Some resistors, capacitors and terminal blocks
Parts:
- C1, C10, C11, C14, C15, C16, C17, C18, C19, C2, C20, C21, C22, C3, C6, C7, C8, C9: footprint ProPrj_Maggy 4.1_2025-02-07-import-fps:C0805 -> Capacitor_SMD:C_0805_2012Metric
- C12, C13, C4, C5: footprint ProPrj_Maggy 4.1_2025-02-07-import-fps:CAP-SMD_BD6.3-L6.6-W6.6-LS7.2-FD -> Capacitor_SMD:C_Elec_6.3x7.7
- CN1: footprint ProPrj_Maggy 4.1_2025-02-07-import-fps:CONN-TH_0430450800 -> Connector_Molex:Molex_Micro-Fit_3.0_43045-0800_2x04_P3.00mm_Horizontal
- CN2: footprint ProPrj_Maggy 4.1_2025-02-07-import-fps:CONN-TH_43045-1000 -> Connector_Molex:Molex_Micro-Fit_3.0_43045-1000_2x05_P3.00mm_Horizontal
- R1, R2, R3, R8, R9: footprint ProPrj_Mag-easyedapro: -> Resistor_SMD:R_0805_2012Metric
- R10, R11, R12, R13, R4, R5, R6, R7: footprint ProPrj_Maggy 4.1_2025-02-07-import-fps:R0805 -> Resistor_SMD:R_0805_2012Metric
- R15, R16, R17, R18: footprint ProPrj_Maggy 4.1_2025-02-07-import-fps:R1206 -> Resistor_SMD:R_1206_3216Metric
- R19, R20, R21, R22, R23, R24: footprint ProPrj_Mag-easyedapro:R0805 -> Resistor_SMD:R_0805_2012Metric
- U1, U10, U2, U9: footprint ProPrj_Maggy 4.1_2025-02-07-import-fps:SOIC-8_L4.9-W3.9-P1.27-LS6.0-BL-EP -> Package_SO:SOIC-8-1EP_3.9x4.9mm_P1.27mm_EP2.41x3.3mm_ThermalVias
Changed lines of the file:
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@@
 			)
 		)
-		(property "Footprint" "ProPrj_Mag-easyedapro:"
+		(property "Footprint" "Resistor_SMD:R_0805_2012Metric"
 			(at 66.04 95.25 0)
 			(hide yes)
@@
 			)
 		)
-		(property "Footprint" "ProPrj_Maggy 4.1_2025-02-07-import-fps:SOIC-8_L4.9-W3.9-P1.27-LS6.0-BL-EP"
+		(property "Footprint" "Package_SO:SOIC-8-1EP_3.9x4.9mm_P1.27mm_EP2.41x3.3mm_ThermalVias"
 			(at 54.61 275.59 0)
 			(hide yes)
@@
 			)
 		)
-		(property "Footprint" "ProPrj_Maggy 4.1_2025-02-07-import-fps:C0805"
+		(property "Footprint" "Capacitor_SMD:C_0805_2012Metric"
 			(at 162.56 234.95 0)
 			(hide yes)
@@
 			)
 		)
-		(property "Footprint" "ProPrj_Maggy 4.1_2025-02-07-import-fps:R1206"
+		(property "Footprint" "Resistor_SMD:R_1206_3216Metric"
 			(at 250.19 278.13 0)
 			(hide yes)
@@
 			)
 		)
-		(property "Footprint" "ProPrj_Maggy 4.1_2025-02-07-import-fps:CONN-TH_0430450800"
+		(property "Footprint" "Connector_Molex:Molex_Micro-Fit_3.0_43045-0800_2x04_P3.00mm_Horizontal"
 			(at 53.34 153.67 0)
 			(hide yes)
@@
 			)
 		)
-		(property "Footprint" "ProPrj_Maggy 4.1_2025-02-07-import-fps:SOIC-8_L4.9-W3.9-P1.27-LS6.0-BL-EP"
+		(property "Footprint" "Package_SO:SOIC-8-1EP_3.9x4.9mm_P1.27mm_EP2.41x3.3mm_ThermalVias"
 			(at 137.16 275.59 0)
 			(hide yes)
@@
 			)
 		)
-		(property "Footprint" "ProPrj_Mag-easyedapro:R0805"
+		(property "Footprint" "Resistor_SMD:R_0805_2012Metric"
 			(at 364.49 66.04 0)
 			(hide yes)
@@
 			)
 		)
-		(property "Footprint" "ProPrj_Maggy 4.1_2025-02-07-import-fps:C0805"
+		(property "Footprint" "Capacitor_SMD:C_0805_2012Metric"
 			(at 78.74 288.29 0)
 			(hide yes)
@@
 			)
 		)
-		(property "Footprint" "ProPrj_Maggy 4.1_2025-02-07-import-fps:R0805"
+		(property "Footprint" "Resistor_SMD:R_0805_2012Metric"
 			(at 83.82 270.51 0)
 			(hide yes)
@@
 			)
 		)
-		(property "Footprint" "ProPrj_Maggy 4.1_2025-02-07-import-fps:R0805"
+		(property "Footprint" "Resistor_SMD:R_0805_2012Metric"
 			(at 166.37 270.51 0)
 			(hide yes)
@@
 			)
 		)
-		(property "Footprint" "ProPrj_Maggy 4.1_2025-02-07-import-fps:R1206"
+		(property "Footprint" "Resistor_SMD:R_1206_3216Metric"
 			(at 330.2 278.13 0)
 			(hide yes)
@@
 			)
 		)
-		(property "Footprint" "ProPrj_Maggy 4.1_2025-02-07-import-fps:C0805"
+		(property "Footprint" "Capacitor_SMD:C_0805_2012Metric"
 			(at 163.83 41.91 0)
 			(hide yes)
@@
 			)
 		)
-		(property "Footprint" "ProPrj_Maggy 4.1_2025-02-07-import-fps:C0805"
+		(property "Footprint" "Capacitor_SMD:C_0805_2012Metric"
 			(at 125.73 76.2 0)
 			(hide yes)
@@
 			)
 		)
-		(property "Footprint" "ProPrj_Maggy 4.1_2025-02-07-import-fps:R0805"
+		(property "Footprint" "Resistor_SMD:R_0805_2012Metric"
 			(at 171.45 82.55 0)
 			(hide yes)
@@
 			)
 		)
-		(property "Footprint" "ProPrj_Maggy 4.1_2025-02-07-import-fps:C0805"
+		(property "Footprint" "Capacitor_SMD:C_0805_2012Metric"
 			(at 289.56 237.49 0)
 			(hide yes)
@@
 			)
 		)
-		(property "Footprint" "ProPrj_Maggy 4.1_2025-02-07-import-fps:C0805"
+		(property "Footprint" "Capacitor_SMD:C_0805_2012Metric"
 			(at 290.83 274.32 0)
 			(hide yes)
@@
 			)
 		)
-		(property "Footprint" "ProPrj_Maggy 4.1_2025-02-07-import-fps:C0805"
+		(property "Footprint" "Capacitor_SMD:C_0805_2012Metric"
 			(at 161.29 288.29 0)
 			(hide yes)
@@
 			)
 		)
-		(property "Footprint" "ProPrj_Maggy 4.1_2025-02-07-import-fps:C0805"
+		(property "Footprint" "Capacitor_SMD:C_0805_2012Metric"
 			(at 388.62 194.31 0)
 			(hide yes)
@@
 			)
 		)
-		(property "Footprint" "ProPrj_Maggy 4.1_2025-02-07-import-fps:R0805"
+		(property "Footprint" "Resistor_SMD:R_0805_2012Metric"
 			(at 86.36 97.79 0)
 			(hide yes)
@@
 			)
 		)
-		(property "Footprint" "ProPrj_Maggy 4.1_2025-02-07-import-fps:C0805"
+		(property "Footprint" "Capacitor_SMD:C_0805_2012Metric"
 			(at 388.62 57.15 0)
 			(hide yes)
@@
 			)
 		)
-		(property "Footprint" "ProPrj_Maggy 4.1_2025-02-07-import-fps:R1206"
+		(property "Footprint" "Resistor_SMD:R_1206_3216Metric"
 			(at 250.19 241.3 0)
 			(hide yes)
@@
 			)
 		)
-		(property "Footprint" "ProPrj_Maggy 4.1_2025-02-07-import-fps:R0805"
+		(property "Footprint" "Resistor_SMD:R_0805_2012Metric"
 			(at 83.82 218.44 0)
 			(hide yes)
@@
 			)
 		)
-		(property "Footprint" "ProPrj_Mag-easyedapro:"
+		(property "Footprint" "Resistor_SMD:R_0805_2012Metric"
 			(at 124.46 128.27 0)
 			(hide yes)
@@
 			)
 		)
-		(property "Footprint" "ProPrj_Mag-easyedapro:R0805"
+		(property "Footprint" "Resistor_SMD:R_0805_2012Metric"
 			(at 222.25 97.79 0)
 			(hide yes)
@@
 			)
 		)
-		(property "Footprint" "ProPrj_Maggy 4.1_2025-02-07-import-fps:SOIC-8_L4.9-W3.9-P1.27-LS6.0-BL-EP"
+		(property "Footprint" "Package_SO:SOIC-8-1EP_3.9x4.9mm_P1.27mm_EP2.41x3.3mm_ThermalVias"
 			(at 138.43 222.25 0)
 			(hide yes)
@@
 			)
 		)
-		(property "Footprint" "ProPrj_Maggy 4.1_2025-02-07-import-fps:R0805"
+		(property "Footprint" "Resistor_SMD:R_0805_2012Metric"
 			(at 102.87 157.48 0)
 			(hide yes)
@@
 			)
 		)
-		(property "Footprint" "ProPrj_Maggy 4.1_2025-02-07-import-fps:C0805"
+		(property "Footprint" "Capacitor_SMD:C_0805_2012Metric"
 			(at 78.74 236.22 0)
 			(hide yes)
@@
 			)
 		)
-		(property "Footprint" "ProPrj_Maggy 4.1_2025-02-07-import-fps:R0805"
+		(property "Footprint" "Resistor_SMD:R_0805_2012Metric"
 			(at 171.45 48.26 0)
 			(hide yes)
@@
 			)
 		)
-		(property "Footprint" "ProPrj_Maggy 4.1_2025-02-07-import-fps:C0805"
+		(property "Footprint" "Capacitor_SMD:C_0805_2012Metric"
 			(at 388.62 91.44 0)
 			(hide yes)
@@
 			)
 		)
-		(property "Footprint" "ProPrj_Maggy 4.1_2025-02-07-import-fps:C0805"
+		(property "Footprint" "Capacitor_SMD:C_0805_2012Metric"
 			(at 388.62 160.02 0)
 			(hide yes)
@@
 			)
 		)
-		(property "Footprint" "ProPrj_Maggy 4.1_2025-02-07-import-fps:C0805"
+		(property "Footprint" "Capacitor_SMD:C_0805_2012Metric"
 			(at 210.82 274.32 0)
 			(hide yes)
@@
 			)
 		)
-		(property "Footprint" "ProPrj_Maggy 4.1_2025-02-07-import-fps:C0805"
+		(property "Footprint" "Capacitor_SMD:C_0805_2012Metric"
 			(at 388.62 125.73 0)
 			(hide yes)
@@
 			)
 		)
-		(property "Footprint" "ProPrj_Maggy 4.1_2025-02-07-import-fps:CONN-TH_43045-1000"
+		(property "Footprint" "Connector_Molex:Molex_Micro-Fit_3.0_43045-1000_2x05_P3.00mm_Horizontal"
 			(at 53.34 173.99 0)
 			(hide yes)
@@
 			)
 		)
-		(property "Footprint" "ProPrj_Mag-easyedapro:"
+		(property "Footprint" "Resistor_SMD:R_0805_2012Metric"
 			(at 124.46 115.57 0)
 			(hide yes)
@@
 			)
 		)
-		(property "Footprint" "ProPrj_Maggy 4.1_2025-02-07-import-fps:C0805"
+		(property "Footprint" "Capacitor_SMD:C_0805_2012Metric"
 			(at 163.83 76.2 0)
 			(hide yes)
@@
 			)
 		)
-		(property "Footprint" "ProPrj_Maggy 4.1_2025-02-07-import-fps:C0805"
+		(property "Footprint" "Capacitor_SMD:C_0805_2012Metric"
 			(at 210.82 237.49 0)
 			(hide yes)
@@
 			)
 		)
-		(property "Footprint" "ProPrj_Maggy 4.1_2025-02-07-import-fps:CAP-SMD_BD6.3-L6.6-W6.6-LS7.2-FD"
+		(property "Footprint" "Capacitor_SMD:C_Elec_6.3x7.7"
 			(at 91.44 288.29 0)
 			(hide yes)
@@
 			)
 		)
-		(property "Footprint" "ProPrj_Maggy 4.1_2025-02-07-import-fps:C0805"
+		(property "Footprint" "Capacitor_SMD:C_0805_2012Metric"
 			(at 125.73 41.91 0)
 			(hide yes)
@@
 			)
 		)
-		(property "Footprint" "ProPrj_Maggy 4.1_2025-02-07-import-fps:CAP-SMD_BD6.3-L6.6-W6.6-LS7.2-FD"
+		(property "Footprint" "Capacitor_SMD:C_Elec_6.3x7.7"
 			(at 91.44 237.49 0)
 			(hide yes)
@@
 			)
 		)
-		(property "Footprint" "ProPrj_Mag-easyedapro:R0805"
+		(property "Footprint" "Resistor_SMD:R_0805_2012Metric"
 			(at 364.49 100.33 0)
 			(hide yes)
@@
 			)
 		)
-		(property "Footprint" "ProPrj_Maggy 4.1_2025-02-07-import-fps:R0805"
+		(property "Footprint" "Resistor_SMD:R_0805_2012Metric"
 			(at 167.64 217.17 0)
 			(hide yes)
@@
 			)
 		)
-		(property "Footprint" "ProPrj_Maggy 4.1_2025-02-07-import-fps:CAP-SMD_BD6.3-L6.6-W6.6-LS7.2-FD"
+		(property "Footprint" "Capacitor_SMD:C_Elec_6.3x7.7"
 			(at 173.99 288.29 0)
 			(hide yes)
@@
 			)
 		)
-		(property "Footprint" "ProPrj_Maggy 4.1_2025-02-07-import-fps:CAP-SMD_BD6.3-L6.6-W6.6-LS7.2-FD"
+		(property "Footprint" "Capacitor_SMD:C_Elec_6.3x7.7"
 			(at 175.26 234.95 0)
 			(hide yes)
@@
 			)
 		)
-		(property "Footprint" "ProPrj_Mag-easyedapro:"
+		(property "Footprint" "Resistor_SMD:R_0805_2012Metric"
 			(at 27.94 114.3 0)
 			(hide yes)
@@
 			)
 		)
-		(property "Footprint" "ProPrj_Maggy 4.1_2025-02-07-import-fps:C0805"
+		(property "Footprint" "Capacitor_SMD:C_0805_2012Metric"
 			(at 76.2 95.25 0)
 			(hide yes)
@@
 			)
 		)
-		(property "Footprint" "ProPrj_Mag-easyedapro:R0805"
+		(property "Footprint" "Resistor_SMD:R_0805_2012Metric"
 			(at 364.49 134.62 0)
 			(hide yes)
@@
 			)
 		)
-		(property "Footprint" "ProPrj_Maggy 4.1_2025-02-07-import-fps:SOIC-8_L4.9-W3.9-P1.27-LS6.0-BL-EP"
+		(property "Footprint" "Package_SO:SOIC-8-1EP_3.9x4.9mm_P1.27mm_EP2.41x3.3mm_ThermalVias"
 			(at 54.61 223.52 0)
 			(hide yes)
@@
 			)
 		)
-		(property "Footprint" "ProPrj_Mag-easyedapro:"
+		(property "Footprint" "Resistor_SMD:R_0805_2012Metric"
 			(at 41.91 97.79 0)
 			(hide yes)
@@
 			)
 		)
-		(property "Footprint" "ProPrj_Mag-easyedapro:R0805"
+		(property "Footprint" "Resistor_SMD:R_0805_2012Metric"
 			(at 364.49 168.91 0)
 			(hide yes)
@@
 			)
 		)
-		(property "Footprint" "ProPrj_Mag-easyedapro:R0805"
+		(property "Footprint" "Resistor_SMD:R_0805_2012Metric"
 			(at 364.49 31.75 0)
 			(hide yes)
@@
 			)
 		)
-		(property "Footprint" "ProPrj_Maggy 4.1_2025-02-07-import-fps:R1206"
+		(property "Footprint" "Resistor_SMD:R_1206_3216Metric"
 			(at 328.93 241.3 0)
 			(hide yes)
