File: Maggy.kicad_sch (KiCad schematic)
At the start: 77 parts, among them CN1 0430450800, CN2 430451000, J1 XY308-2.54-2P, J2 XY308-2.54-2P, J3 XY308-2.54-2P, J4 XY308-2.54-2P, J5 X6511FV-24-C85D32, J6 X6511FV-24-C85D32, U1 CH224K, U10 INA214AIDCKR, U11 Socket for Teensy 4.1 (2x 1x2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, U12 INA214AIDCKR, U13 INA214AIDCKR, U14 TMAG5170A2DGKR, U15 TMAG5170A2DGKR, U16 TMAG5170A2DGKR, U17 TMAG5170A2DGKR, U18 TMAG5170A2DGKR, U2 A4950ELJTR-T, U3 A4950ELJTR-T, U4 A4950ELJTR-T, U5 A4950ELJTR-T, U6 TLV2372, U7 LM1117S-3.3, U8 LM1117S-5.0, U9 INA214AIDCKR

Commit message: chore: remove incorrectly labelled nets, update tracks missing nets
Connections:
- net 1V65 renamed +1V65
- no-connect marks 41 -> 89
Changed lines of the file:
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@@
 	)
 	(no_connect
+		(at 295.91 190.5)
+	)
+	(no_connect
+		(at 295.91 160.02)
+	)
+	(no_connect
+		(at 229.87 177.8)
+	)
+	(no_connect
 		(at 259.08 125.73)
 	)
 	(no_connect
+		(at 295.91 195.58)
+	)
+	(no_connect
 		(at 157.48 134.62)
 	)
@@
 	)
 	(no_connect
+		(at 295.91 170.18)
+	)
+	(no_connect
+		(at 295.91 142.24)
+	)
+	(no_connect
+		(at 229.87 185.42)
+	)
+	(no_connect
 		(at 53.34 64.77)
 	)
@@
 	)
 	(no_connect
+		(at 295.91 149.86)
+	)
+	(no_connect
+		(at 295.91 175.26)
+	)
+	(no_connect
 		(at 290.83 86.36)
 	)
@@
 	)
 	(no_connect
+		(at 295.91 182.88)
+	)
+	(no_connect
 		(at 234.95 113.03)
 	)
 	(no_connect
+		(at 229.87 157.48)
+	)
+	(no_connect
+		(at 229.87 142.24)
+	)
+	(no_connect
+		(at 229.87 149.86)
+	)
+	(no_connect
+		(at 229.87 180.34)
+	)
+	(no_connect
 		(at 234.95 91.44)
 	)
 	(no_connect
+		(at 229.87 198.12)
+	)
+	(no_connect
 		(at 290.83 93.98)
 	)
@@
 	)
 	(no_connect
+		(at 229.87 147.32)
+	)
+	(no_connect
 		(at 290.83 96.52)
 	)
 	(no_connect
+		(at 229.87 144.78)
+	)
+	(no_connect
 		(at 234.95 66.04)
 	)
 	(no_connect
+		(at 229.87 187.96)
+	)
+	(no_connect
+		(at 229.87 160.02)
+	)
+	(no_connect
+		(at 229.87 154.94)
+	)
+	(no_connect
+		(at 229.87 139.7)
+	)
+	(no_connect
+		(at 229.87 193.04)
+	)
+	(no_connect
+		(at 295.91 147.32)
+	)
+	(no_connect
+		(at 295.91 139.7)
+	)
+	(no_connect
 		(at 290.83 91.44)
 	)
 	(no_connect
+		(at 295.91 177.8)
+	)
+	(no_connect
+		(at 295.91 180.34)
+	)
+	(no_connect
 		(at 290.83 88.9)
 	)
@@
 	)
 	(no_connect
+		(at 229.87 152.4)
+	)
+	(no_connect
 		(at 172.72 132.08)
 	)
@@
 	)
 	(no_connect
+		(at 229.87 167.64)
+	)
+	(no_connect
 		(at 234.95 107.95)
 	)
 	(no_connect
+		(at 295.91 162.56)
+	)
+	(no_connect
 		(at 234.95 110.49)
 	)
 	(no_connect
+		(at 295.91 152.4)
+	)
+	(no_connect
+		(at 229.87 190.5)
+	)
+	(no_connect
+		(at 295.91 193.04)
+	)
+	(no_connect
 		(at 234.95 40.64)
 	)
 	(no_connect
+		(at 229.87 172.72)
+	)
+	(no_connect
 		(at 290.83 58.42)
 	)
@@
 	)
 	(no_connect
+		(at 295.91 167.64)
+	)
+	(no_connect
 		(at 234.95 104.14)
 	)
 	(no_connect
+		(at 229.87 162.56)
+	)
+	(no_connect
+		(at 295.91 198.12)
+	)
+	(no_connect
+		(at 229.87 182.88)
+	)
+	(no_connect
 		(at 234.95 101.6)
 	)
@@
 	)
 	(no_connect
+		(at 295.91 157.48)
+	)
+	(no_connect
+		(at 295.91 187.96)
+	)
+	(no_connect
 		(at 234.95 118.11)
 	)
 	(no_connect
+		(at 229.87 170.18)
+	)
+	(no_connect
+		(at 295.91 154.94)
+	)
+	(no_connect
+		(at 295.91 185.42)
+	)
+	(no_connect
 		(at 255.27 125.73)
 	)
 	(no_connect
+		(at 295.91 144.78)
+	)
+	(no_connect
+		(at 229.87 175.26)
+	)
+	(no_connect
+		(at 295.91 165.1)
+	)
+	(no_connect
 		(at 290.83 34.29)
 	)
@@
 	)
 	(no_connect
+		(at 229.87 165.1)
+	)
+	(no_connect
+		(at 229.87 195.58)
+	)
+	(no_connect
+		(at 295.91 172.72)
+	)
+	(no_connect
 		(at 290.83 107.95)
 	)
@@
 		)
 	)
-	(global_label "1V65"
+	(global_label "+1V65"
 		(shape input)
 		(at 243.84 275.59 270)
@@
 		)
 		(property "Intersheetrefs" "${INTERSHEET_REFS}"
-			(at 243.84 283.2923 90)
+			(at 243.84 284.8647 90)
 			(hide yes)
 			(show_name no)
@@
 		)
 	)
-	(global_label "1V65"
+	(global_label "+1V65"
 		(shape input)
 		(at 307.34 242.57 270)
@@
 		)
 		(property "Intersheetrefs" "${INTERSHEET_REFS}"
-			(at 307.34 250.2723 90)
+			(at 307.34 251.8447 90)
 			(hide yes)
 			(show_name no)
@@
 		)
 	)
-	(global_label "1V65"
+	(global_label "+1V65"
 		(shape output)
 		(at 175.26 113.03 0)
@@
 		)
 		(property "Intersheetrefs" "${INTERSHEET_REFS}"
-			(at 182.9623 113.03 0)
+			(at 184.5347 113.03 0)
 			(hide yes)
 			(show_name no)
@@
 		)
 	)
-	(global_label "1V65"
+	(global_label "+1V65"
 		(shape input)
 		(at 243.84 242.57 270)
@@
 		)
 		(property "Intersheetrefs" "${INTERSHEET_REFS}"
-			(at 243.84 250.2723 90)
+			(at 243.84 251.8447 90)
 			(hide yes)
 			(show_name no)
@@
 		)
 	)
-	(global_label "1V65"
+	(global_label "+1V65"
 		(shape input)
 		(at 307.34 275.59 270)
@@
 		)
 		(property "Intersheetrefs" "${INTERSHEET_REFS}"
-			(at 307.34 283.2923 90)
+			(at 307.34 284.8647 90)
 			(hide yes)
 			(show_name no)
@@
 		(in_pos_files yes)
 		(dnp no)
-		(fields_autoplaced yes)
 		(property "Reference" "U6"
 			(at 165.1 102.87 0)
@@
 		)
 		(property "Footprint" "Package_SO:SOIC-8_3.9x4.9mm_P1.27mm"
-			(at 165.1 113.03 0)
+			(at 165.354 120.396 0)
+			(hide yes)
 			(show_name no)
 			(do_not_autoplace no)
